File: Docs.sch (KiCad schematic (older format))
At the start: 0 parts

Commit message: Submitted to JLCPCB
Connections:
- wire segments 259 -> 250
Other:
- note added: "Apple II Registers:\n C0XF: ROM bank\n C0XB: Vblank (high bit set if blanking, cleared o.w.)\n C0XA: Read current video byte\n C0X1: Argument/result register\n C0X0: Command/Status register\n\nAVR Registers:\n X1: Argument/result register\n X0: Command/Status register (done, rx, 111111)\n\nMouse Entry Vector Table:\n 19: INITMOUSE: Reset mouse clamps, position\n 18: HOMEMOUSE: Set mouse to top-le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"
- note added: "Commands to AVR:\n FF: SW_RESET\n\n E3: GET_IRQSTATE\n E2: SET_MODE\n E1: INIT_VBL\n E0: INIT_MOUSE\n\n C1: GO_CLEAR (pos)\n C0: GO_HOME (pos)\n\n 83: SET_HI\n 82: SET_LO\n 81: GET_HI\n 80: GET_LO\n\n 53: SET_Y0 (clamp)\n 52: SET_Y1 (clamp)\n 51: SET_X0 (clamp)\n 50: SET_X1 (clamp)\n 41: SET_Y (pos)\n 40: SET_X (pos)\n\n 13: GET_Y0 (clamp)\n 12: GET_Y1 (clamp)\n 11: GET_X0 (clamp)\n 10: GET_X1 (c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"
- note added: "R~CS~ = ~CSEN & (IOSEL | (IOSTRB & IOROMEN))~\nR~OE~ = ~R~W\n\nROMA[15:12] = Bank[4:1]\nROMA[11] = IOSEL ? 0 : Bank[0]\nD[7:0] = (~DEVSEL~ | ~CSEN~ | ~R~W | AVidSEL) ? 8’bZ :\n ACmdStatusSEL ? {CmdDone, CmdRX, ArgRX, 5’h1F} :\n AArgResSEL ? ArgRes[7:0] :\n AVBlSEL ? (VBl ? 0x80 : 0x00)\n\nRAD[7:0] = ~RRD~ ? 8’bZ : RDR[7:0]\nRAR[7:0] = RAD[7:0] @ ALE\nRDR[7:0] = (RCmdStatSEL & ~S3~ & ~RDRSet~) ? C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"
- note added: "S[2:0] = (S == 0) ? 0 : (~Q3~ & PHI1) ? 7 : S+1 @ C7M\nCSEN = S1 | S2 | S3 @ C7M\n\nABankSEL = (A==C0XF) & DEVSEL @ C7M in S7\nAVBlSEL = (A==C0XB) & DEVSEL @ C7M in S7\nAVidSEL = (A==C0XA) & DEVSEL @ C7M in S7\nAArgResSEL = (A==C0X1) & DEVSEL @ C7M in S7\nACmdStatSEL = (A==C0X0) & DEVSEL @ C7M in S7\n\nRArgResSEL = ALE & RA==XXX1\nRCmdStatSEL = ALE & RA==XXX0\n\nIOROMEN = (A==XFFF/X7FF & IOSTRB) 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"
- note removed: "AVR Registers:\n XX0A: Read current video byte\n XX01: Result register\n XX00: Command/Status register\n\nCommands to AVR:\n FF: Software Reset\n 5F: SET_Y0H (clamp)\n 5E: SET_Y0L (clamp)\n 5D: SET_Y1H (clamp)\n 5C: SET_Y1L (clamp)\n 5B: SET_X0H (clamp)\n 5A: SET_X0L (clamp)\n 59: SET_X1H (clamp)\n 58: SET_X1L (clamp)\n 57: SET_YH (pos)\n 56: SET_YL (pos)\n 55: SET_XH (pos)\n 54: SET_XL (pos)\n 5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"
- note removed: "Apple II Registers:\n C0XF: ROM bank (4-bit)\n C0XB: Vblank (8X if blanking, 0X o.w.)\n C0XA: Read current video byte\n C0X1: Result register\n C0X0: Command/Status register\n\nMouse Entry Vector Table:\n 19: INITMOUSE: Reset mouse clamps, position\n 18: HOMEMOUSE: Set mouse to top-left of camp\n 17: CLAMPMOUSE: Bound mouse in a window\n 16: POSMOUSE: Set mouse position\n 15: CLEARMOUSE: Clear mo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"
- note removed: "PHI1"
- note removed: "R~CS~ = ~CSEN & (IOSEL | (IOSTRB & IOROMEN))~\nR~OE~ = ~R~W\n\nA[7:0] = ~AOE~ ? 8’bZ : RAR[7:0]\nD[7:0] = (~DEVSEL~ | ~CSEN~ | ~R~W | AVidSEL) ? 8’bZ :\n ACmdStatusSEL ? {CmdDone, 7’b7F} :\n AArgResHSEL ? ArgResH[7:0] :\n AArgResLSEL ? ArgResL[7:0] :\n AVBlSEL ? (VBl ? 0x80 : 0x00)\n\nRAD[7:0] = ~RRD~ ? 8’bZ : RDR[7:0]\nRAR[7:0] = RAD[7:0] @ ALE\nRDR[7:0] = (RCmdStatSEL & ~S3~ & ~RDRSet~) ? Cmd[7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"
- note removed: "S[2:0] = (S == 0) ? 0 : (~Q3~ & PHI1) ? 7 : S+1 @ C7M\nCSEN = S1 | S2 | S3 @ C7M\n\nABankSEL = (A==C0XF) & DEVSEL @ C7M in S7\nAVBlSEL = (A==C0XB) & DEVSEL @ C7M in S7\nAVidSEL = (A==C0XA) & DEVSEL @ C7M in S7\nAArgResHSEL = (A==C0X3) & DEVSEL @ C7M in S7\nAArgResLSEL = (A==C0X2) & DEVSEL @ C7M in S7\nACmdStatSEL = (A==C0X0) & DEVSEL @ C7M in S7\n\nRArgResHSEL = ALE & RA==XXX3\nRArgResLSEL = ALE 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"

Commit message: Adapter stuff, avr
Changed lines of the file:
@@
 Comment4 ""
 $EndDescr
-Text Notes 4300 1250 0    40   ~ 0
-S7
 Text Notes 1600 1400 2    50   ~ 0
 PHI0
@@
 	4450 1300 6550 1300
 Text Notes 1900 1250 0    40   ~ 0
-S3
-Text Notes 6700 1250 0    40   ~ 0
-S4
+S6
 Text Notes 6100 1250 0    40   ~ 0
-S3
-Text Notes 5500 1250 0    40   ~ 0
-S2
-Text Notes 4900 1250 0    40   ~ 0
-S1
-Text Notes 3700 1250 0    40   ~ 0
 S6
-Text Notes 3100 1250 0    40   ~ 0
-S5
 Wire Wire Line
 	3500 1150 3800 1150
-Text Notes 2500 1250 0    40   ~ 0
-S4
 Wire Wire Line
 	2000 1250 2300 1250
@@
 	6500 1150 6800 1150
 Text Notes 8500 1250 0    40   ~ 0
-S7
+S3
 Wire Wire Line
 	6550 1300 6550 1400
@@
 	6550 1400 8650 1400
 Text Notes 7900 1250 0    40   ~ 0
-S6
+S2
 Text Notes 7300 1250 0    40   ~ 0
-S5
+S1
 Wire Wire Line
 	7700 1150 8000 1150
 Text Notes 6700 1250 0    40   ~ 0
-S4
+S7
 Wire Wire Line
 	8000 1150 8000 1250
@@
 Text Notes 8250 5950 0    50   ~ 0
 Commands to AVR:\n  FF: SW_RESET\n\n  E3: GET_IRQSTATE\n  E2: SET_MODE\n  E1: INIT_VBL\n  E0: INIT_MOUSE\n\n  C1: GO_CLEAR (pos)\n  C0: GO_HOME (pos)\n\n  83: SET_HI\n  82: SET_LO\n  81: GET_HI\n  80: GET_LO\n\n  53: SET_Y0 (clamp)\n  52: SET_Y1 (clamp)\n  51: SET_X0 (clamp)\n  50: SET_X1 (clamp)\n  41: SET_Y (pos)\n  40: SET_X (pos)\n\n  13: GET_Y0 (clamp)\n  12: GET_Y1 (clamp)\n  11: GET_X0 (clamp)\n  10: GET_X1 (clamp)\n  01: GET_Y (pos)\n  00: GET_X (pos)
+Text Notes 5500 1250 0    40   ~ 0
+S5
+Text Notes 4900 1250 0    40   ~ 0
+S4
+Text Notes 4300 1250 0    40   ~ 0
+S3
+Text Notes 3700 1250 0    40   ~ 0
+S2
+Text Notes 3100 1250 0    40   ~ 0
+S1
+Text Notes 2500 1250 0    40   ~ 0
+S7
 $EndSCHEMATC
