File: Mouserial.sch (KiCad schematic (older format))
At the start: 49 parts, among them J1 AppleIIBus, J2 JTAG, J3 AVRISP, J4 USBmicroB, J5 PS/2, U1 EPM7128SL84, U2 ATmega8515L-8JU, U3 39SF010, U4 CH340G, Y1 12M

Commit message: Submitted to JLCPCB
Parts:
- removed C17: 33u, stdpads:CP_EIA-3528, symbol Device:CP_Small
- removed FD1, FD2, FD3, FD4, FD5: Fiducial, stdpads:Fiducial, symbol Mechanical:MountingHole
- removed J5: PS/2, stdpads:IDC_SMD_2x03_P2.54mm_Vertical, symbol Connector_Generic:Conn_02x03_Odd_Even
- removed JP1: Pgm, Connector_PinHeader_2.54mm:PinHeader_1x02_P2.54mm_Vertical_SMD_Pin1Right, symbol Device:Jumper_NO_Small
- added C17, C22: 100n, stdpads:C_0805, symbol Device:C_Small
- added C23: 33u, stdpads:CP_EIA-3528, symbol Device:CP_Small
- added FID1, FID2, FID3, FID4, FID5: Fiducial, stdpads:Fiducial, symbol Mechanical:Fiducial
- added J5: PS/2, stdpads:IDC_SMD_2x04_P2.54mm_Vertical, symbol Connector_Generic:Conn_02x04_Odd_Even
- added JP1: P/K, Connector_PinHeader_2.54mm:PinHeader_2x02_P2.54mm_Vertical_SMD, symbol Connector_Generic:Conn_02x02_Odd_Even
- added R10, R8, R9: 4k7, stdpads:R_0805, symbol Device:R_Small
- J4: footprint Connector_USB:USB_Micro-B_Molex_47346-0001 -> stdpads:USB_Micro-B_Amphenol_10118192-0001
- R1: value 1k -> 4k7
- R2, R3: value 10k -> 4k7
- R7: value 100 -> 4k7
- U4: footprint Package_SO:SOIC-16_3.9x9.9mm_P1.27mm -> stdpads:SOIC-16_3.9mm
- Y1: footprint Crystal:Crystal_SMD_HC49-SD -> stdpads:Crystal_HC49-SMD
Connections:
- net +5V: now also R7.1, C17.1, C23.1, J5.3 (Pin_3), R10.1, R8.1, R9.1
- net -12V: now also C22.2
- net -5V: now also C17.2, C22.1
- net A11: no longer U3.25 (A11)
- net A12: now also U1.52 (I/O)
- net A13: now also U1.51 (I/O)
- net A14: now also U1.50 (I/O)
- net A15: now also U1.39 (I/O/NC)
- net GND: now also U1.19 (GND), U1.32 (GND), C23.2, J5.2 (Pin_2), J5.5 (Pin_5), J5.6 (Pin_6), JP1.4 (Pin_4); no longer U4.15 (R232)
- net PHI1: no longer R7.2
- net ROMA16: now also R7.2
- net RXD: now also U4.2 (TXD); no longer U4.3 (RXD)
- net R~RST~: now also JP1.1 (Pin_1)
- net TXD: now also U4.3 (RXD); no longer U4.2 (TXD)
- net ~INH~: now also U1.81 (I/O)
- net ~KMode~: now reaches U1.40 (I/O)
- net ~KMode~: now also JP1.3 (Pin_3), R10.2
- net ROMA11: now reaches U1.68 (I/O)
- net ROMA11: now also U3.25 (A11)
- net at C21.2: now also JP1.2 (Pin_2)
- net MDat: now reaches U2.16 (PD4)
- net MDat: now also R2.2, J5.7 (Pin_7)
- removed net PHI1r: R7.1, U1.81 (I/O)
- net PS2_Clk renamed KClk
- net KClk: now also J5.4 (Pin_4), R9.2; no longer R3.2
- net PS2_Dat renamed KDat
- net KDat: now also J5.8 (Pin_8), R8.2; no longer R2.2
- net ~RI~: no longer names the net of U4.11 (~RI)
- net ~RI~: no longer U2.27 (PC3)
- net ~SYNC~: no longer names the net of U1.16 (I/O)
- net ~SYNC~: no longer J1.19 (Pin_19)
- new net MClk: J5.1 (Pin_1), R3.2, U2.27 (PC3)
- new net VIDSYNC: J1.19 (Pin_19)
- no-connect marks 12 -> 8
Other:
- note added: "ROM mode select"
- note added: "RS232"
- note added: "RS232 Serial"
- note removed: "More\nRS232"
- note removed: "Serial"
- moved on the sheet: C21, R1, U2

Commit message: Adapter stuff, avr
Parts:
- C1, C12, C13, C14, C15, C17, C2, C22: value 100n -> 2u2
- C19, C21: value 100n -> 10n
- R4: value 100 -> 15
Changed lines of the file:
@@
 P 5800 5850
 F 0 "C1" H 5850 5900 50  0000 L CNN
-F 1 "100n" H 5850 5800 50  0000 L CNN
+F 1 "2u2" H 5850 5800 50  0000 L CNN
 F 2 "stdpads:C_0805" H 5800 5850 50  0001 C CNN
 F 3 "~" H 5800 5850 50  0001 C CNN
@@
 P 6200 5850
 F 0 "C2" H 6250 5900 50  0000 L CNN
-F 1 "100n" H 6250 5800 50  0000 L CNN
+F 1 "2u2" H 6250 5800 50  0000 L CNN
 F 2 "stdpads:C_0805" H 6200 5850 50  0001 C CNN
 F 3 "~" H 6200 5850 50  0001 C CNN
@@
 P 4650 7100
 F 0 "C14" H 4700 7150 50  0000 L CNN
-F 1 "100n" H 4700 7050 50  0000 L CNN
+F 1 "2u2" H 4700 7050 50  0000 L CNN
 F 2 "stdpads:C_0805" H 4650 7100 50  0001 C CNN
 F 3 "~" H 4650 7100 50  0001 C CNN
@@
 P 4650 7400
 F 0 "C15" H 4700 7450 50  0000 L CNN
-F 1 "100n" H 4700 7350 50  0000 L CNN
+F 1 "2u2" H 4700 7350 50  0000 L CNN
 F 2 "stdpads:C_0805" H 4650 7400 50  0001 C CNN
 F 3 "~" H 4650 7400 50  0001 C CNN
@@
 P 4250 7100
 F 0 "C12" H 4300 7150 50  0000 L CNN
-F 1 "100n" H 4300 7050 50  0000 L CNN
+F 1 "2u2" H 4300 7050 50  0000 L CNN
 F 2 "stdpads:C_0805" H 4250 7100 50  0001 C CNN
 F 3 "~" H 4250 7100 50  0001 C CNN
@@
 P 4250 7400
 F 0 "C13" H 4300 7450 50  0000 L CNN
-F 1 "100n" H 4300 7350 50  0000 L CNN
+F 1 "2u2" H 4300 7350 50  0000 L CNN
 F 2 "stdpads:C_0805" H 4250 7400 50  0001 C CNN
 F 3 "~" H 4250 7400 50  0001 C CNN
@@
 P 9550 5200
 F 0 "C19" H 9600 5250 50  0000 L CNN
-F 1 "100n" H 9600 5150 50  0000 L CNN
+F 1 "10n" H 9600 5150 50  0000 L CNN
 F 2 "stdpads:C_0805" H 9550 5200 50  0001 C CNN
 F 3 "~" H 9550 5200 50  0001 C CNN
@@
 Text Label 5350 3700 0    50   ~ 0
 VBl1
-$Comp
-L stdparts:EPM7128SL84 U1
-U 1 1 5CBA3E53
-P 4600 2900
-F 0 "U1" H 4600 2950 50  0000 C CNN
-F 1 "EPM7128SL84" H 4600 2850 50  0000 C CNN
-F 2 "stdpads:PLCC-84_SMDSocket" H 4450 3100 50  0001 C CNN
-F 3 "" H 4450 3100 50  0001 C CNN
-	1    4600 2900
-	-1   0    0    -1
-$EndComp
 Text Label 3850 3100 2    50   ~ 0
 D7
@@
 Wire Wire Line
 	4250 7250 4250 7300
-$Comp
-L Device:R_Small R4
-U 1 1 5D6D5B73
-P 2800 4150
-F 0 "R4" V 2650 4150 50  0000 C CNN
-F 1 "100" V 2750 4150 50  0000 C BNN
-F 2 "stdpads:R_0805" H 2800 4150 50  0001 C CNN
-F 3 "~" H 2800 4150 50  0001 C CNN
-	1    2800 4150
-	0    1    1    0
-$EndComp
 Text Label 2900 4450 0    50   ~ 0
 Q3r
@@
 Text Label 6900 2250 2    50   ~ 0
 TCK
-Wire Wire Line
-	4950 900  4850 900
-Connection ~ 4250 900
-Connection ~ 4850 900
-Wire Wire Line
-	4850 900  4750 900
-Connection ~ 4750 900
-Wire Wire Line
-	4750 900  4650 900
-Connection ~ 4650 900
-Wire Wire Line
-	4650 900  4550 900
-Connection ~ 4550 900
-Wire Wire Line
-	4550 900  4450 900
-Connection ~ 4450 900
-Wire Wire Line
-	4450 900  4350 900
-Connection ~ 4350 900
-Wire Wire Line
-	4350 900  4250 900
 Text Label 6900 2350 2    50   ~ 0
 TDO
@@
 Entry Wire Line
 	6600 2050 6700 1950
-Wire Wire Line
-	4750 5000 4650 5000
-Connection ~ 4650 5000
-Wire Wire Line
-	4650 5000 4550 5000
-Connection ~ 4550 5000
-Wire Wire Line
-	4550 5000 4450 5000
-Connection ~ 4450 5000
-Wire Wire Line
-	4450 5000 4350 5000
-Connection ~ 4350 5000
-Wire Wire Line
-	4350 5000 4250 5000
 Text Label 10150 2500 0    50   ~ 0
 MOSI
@@
 P 9950 1600
 F 0 "C21" V 9721 1600 50  0000 C CNN
-F 1 "100n" V 9812 1600 50  0000 C CNN
+F 1 "10n" V 9812 1600 50  0000 C CNN
 F 2 "stdpads:C_0805" H 9950 1600 50  0001 C CNN
 F 3 "~" H 9950 1600 50  0001 C CNN
@@
 L power:GND #PWR0131
 U 1 1 5D59E16D
-P 10250 800
-F 0 "#PWR0131" H 10250 550 50  0001 C CNN
-F 1 "GND" H 10250 650 50  0000 C CNN
-F 2 "" H 10250 800 50  0001 C CNN
-F 3 "" H 10250 800 50  0001 C CNN
-	1    10250 800
-	-1   0    0    1
-$EndComp
-Wire Wire Line
-	9950 800  10250 800
+P 10250 1000
+F 0 "#PWR0131" H 10250 750 50  0001 C CNN
+F 1 "GND" H 10250 850 50  0000 C CNN
+F 2 "" H 10250 1000 50  0001 C CNN
+F 3 "" H 10250 1000 50  0001 C CNN
+	1    10250 1000
+	1    0    0    -1
+$EndComp
 Wire Wire Line
 	9450 1000 9150 1000
@@
 Text Notes 6450 4250 2    50   ~ 0
 ROM mode select
-Connection ~ 4250 5000
-Wire Wire Line
-	4750 5000 4850 5000
-Connection ~ 4750 5000
-Connection ~ 4850 5000
-Wire Wire Line
-	4850 5000 4950 5000
 Wire Wire Line
 	9350 1600 9150 1600
@@
 Wire Wire Line
 	10250 1000 10250 800
-Connection ~ 10250 800
 Text Label 6900 3050 2    50   ~ 0
 KDat
@@
 P 5050 7400
 F 0 "C17" H 5100 7450 50  0000 L CNN
-F 1 "100n" H 5100 7350 50  0000 L CNN
+F 1 "2u2" H 5100 7350 50  0000 L CNN
 F 2 "stdpads:C_0805" H 5050 7400 50  0001 C CNN
 F 3 "~" H 5050 7400 50  0001 C CNN
@@
 P 4450 7550
 F 0 "C22" V 4300 7550 50  0000 C BNN
-F 1 "100n" V 4350 7550 50  0000 C CNN
+F 1 "2u2" V 4350 7550 50  0000 C CNN
 F 2 "stdpads:C_0805" H 4450 7550 50  0001 C CNN
 F 3 "~" H 4450 7550 50  0001 C CNN
@@
 NoConn ~ 8650 5800
 NoConn ~ 5350 1500
+Connection ~ 10250 1000
+Wire Wire Line
+	9950 800  10250 800
+Connection ~ 4850 5000
+Connection ~ 4750 5000
+Wire Wire Line
+	4850 5000 4950 5000
+Wire Wire Line
+	4750 5000 4850 5000
+Connection ~ 4250 5000
+Wire Wire Line
+	4350 5000 4250 5000
+Connection ~ 4350 5000
+Connection ~ 4450 5000
+Wire Wire Line
+	4450 5000 4350 5000
+Wire Wire Line
+	4550 5000 4450 5000
+Connection ~ 4550 5000
+Connection ~ 4650 5000
+Wire Wire Line
+	4650 5000 4550 5000
+Wire Wire Line
+	4750 5000 4650 5000
+Wire Wire Line
+	4350 900  4250 900
+Connection ~ 4350 900
+Connection ~ 4450 900
+Wire Wire Line
+	4450 900  4350 900
+Wire Wire Line
+	4550 900  4450 900
+Connection ~ 4550 900
+Connection ~ 4650 900
+Wire Wire Line
+	4650 900  4550 900
+Wire Wire Line
+	4750 900  4650 900
+Connection ~ 4750 900
+Connection ~ 4850 900
+Connection ~ 4250 900
+Wire Wire Line
+	4850 900  4750 900
+Wire Wire Line
+	4950 900  4850 900
+$Comp
+L stdparts:EPM7128SL84 U1
+U 1 1 5CBA3E53
+P 4600 2900
+F 0 "U1" H 4600 2950 50  0000 C CNN
+F 1 "EPM7128SL84" H 4600 2850 50  0000 C CNN
+F 2 "stdpads:PLCC-84_SMDSocket" H 4450 3100 50  0001 C CNN
+F 3 "" H 4450 3100 50  0001 C CNN
+	1    4600 2900
+	-1   0    0    -1
+$EndComp
+$Comp
+L Device:R_Small R4
+U 1 1 5D6D5B73
+P 2800 4150
+F 0 "R4" V 2650 4150 50  0000 C CNN
+F 1 "15" V 2750 4150 50  0000 C BNN
+F 2 "stdpads:R_0805" H 2800 4150 50  0001 C CNN
+F 3 "~" H 2800 4150 50  0001 C CNN
+	1    2800 4150
+	0    1    1    0
+$EndComp
 Wire Bus Line
 	5700 3600 5700 5200
