File: adapter-keymouse/mouserial-keymouse.sch (KiCad schematic (older format))
At the start: 13 parts, among them J1 Mouserial, J2 Mouse, J3 Keybd

Commit message: Adapter stuff, avr
Parts:
- J1: footprint Connector_PinHeader_1.27mm:PinHeader_1x08_P1.27mm_Vertical -> stdpads:IDC_SMD_2x04_P2.54mm_Vertical
Changed lines of the file:
@@
 F 0 "J1" H 4150 4517 50  0000 C CNN
 F 1 "Mouserial" H 4150 4426 50  0000 C CNN
-F 2 "Connector_PinHeader_1.27mm:PinHeader_1x08_P1.27mm_Vertical" H 4100 4200 50  0001 C CNN
+F 2 "stdpads:IDC_SMD_2x04_P2.54mm_Vertical" H 4100 4200 50  0001 C CNN
 F 3 "~" H 4100 4200 50  0001 C CNN
 	1    4100 4200
@@
 $EndComp
 $Comp
-L power:GND #PWR?
+L power:GND #PWR0106
 U 1 1 5D3291B1
 P 3950 2950
-F 0 "#PWR?" H 3950 2700 50  0001 C CNN
+F 0 "#PWR0106" H 3950 2700 50  0001 C CNN
 F 1 "GND" H 3950 2800 50  0000 C CNN
 F 2 "" H 3950 2950 50  0001 C CNN
@@
 $EndComp
 $Comp
-L power:GND #PWR?
+L power:GND #PWR0107
 U 1 1 5D329649
 P 3950 3450
-F 0 "#PWR?" H 3950 3200 50  0001 C CNN
+F 0 "#PWR0107" H 3950 3200 50  0001 C CNN
 F 1 "GND" H 3950 3300 50  0000 C CNN
 F 2 "" H 3950 3450 50  0001 C CNN
@@
 $EndComp
 $Comp
-L power:GND #PWR?
+L power:GND #PWR0108
 U 1 1 5D329A44
 P 4650 3450
-F 0 "#PWR?" H 4650 3200 50  0001 C CNN
+F 0 "#PWR0108" H 4650 3200 50  0001 C CNN
 F 1 "GND" H 4650 3300 50  0000 C CNN
 F 2 "" H 4650 3450 50  0001 C CNN
@@
 $EndComp
 $Comp
-L power:GND #PWR?
+L power:GND #PWR0109
 U 1 1 5D329D95
 P 4650 2950
-F 0 "#PWR?" H 4650 2700 50  0001 C CNN
+F 0 "#PWR0109" H 4650 2700 50  0001 C CNN
 F 1 "GND" H 4650 2800 50  0000 C CNN
 F 2 "" H 4650 2950 50  0001 C CNN
