File: adapter-mouse/mouserial-mouse.sch (KiCad schematic (older format))
At the start: 12 parts, among them J1 Mouserial, J2 Mouse

Commit message: Adapter stuff, avr
Parts:
- J1: footprint Connector_PinHeader_2.54mm:PinHeader_1x08_P2.54mm_Vertical -> stdpads:IDC_SMD_2x04_P2.54mm_Vertical
Changed lines of the file:
@@
 F 0 "J1" H 4150 4517 50  0000 C CNN
 F 1 "Mouserial" H 4150 4426 50  0000 C CNN
-F 2 "Connector_PinHeader_2.54mm:PinHeader_1x08_P2.54mm_Vertical" H 4100 4200 50  0001 C CNN
+F 2 "stdpads:IDC_SMD_2x04_P2.54mm_Vertical" H 4100 4200 50  0001 C CNN
 F 3 "~" H 4100 4200 50  0001 C CNN
 	1    4100 4200
